File: DevTermCaseTemp.kicad_pcb (KiCad board)
At the start: 2 copper layers, 98.2 x 77 mm, 1 part, among them J1 miniPCIe

Commit message: Update README
Connections:
- J1 pad 11: Net-(J1-Pad11) -> GND
- J1 pad 21: Net-(J1-Pad11) -> GND
- J1 pad 27: Net-(J1-Pad11) -> GND
- J1 pad 33: Net-(J1-Pad11) -> GND
- J1 pad 39: Net-(J1-Pad11) -> GND
- J1 pad 5: Net-(J1-Pad11) -> GND
