File: DevTermCaseTemp.kicad_pcb (KiCad board)
At the start: 2 copper layers, 98.2 x 77 mm, 1 part, among them J1 miniPCIe

Commit message: Update the symbol of mPCIE port
Parts:
- J1: value miniPCIe -> DevTermExtPort
Connections:
- J1 pad 17: unconnected-(J1-Pad17) -> (no net)
- J1 pad 19: unconnected-(J1-Pad19) -> (no net)
- J1 pad 45: unconnected-(J1-Pad45) -> GND
- J1 pad 47: unconnected-(J1-Pad47) -> (no net)
- J1 pad 49: unconnected-(J1-Pad49) -> (no net)
- J1 pad 51: unconnected-(J1-Pad51) -> GND
